Commit message: Added URDF gazebo meta tags

File: src/turtle/urdf/turtle.urdf (robot description, URDF)
Before this commit: robot turtle, 5 links, 4 joints
Links:
- link base_link: geometry collision box size=0.6 0.3 0.3; visual box size=0.6 0.3 0.3
- link front_caster: geometry collision box size=0.1 0.1 0.3; visual box size=0.1 0.1 0.3
- link front_wheel: geometry collision cylinder length=0.05 radius=0.035; visual cylinder length=0.05 radius=0.035
- link right_wheel: geometry collision cylinder length=0.05 radius=0.035; visual cylinder length=0.05 radius=0.035

Commit message: Fixed bug: inertia -> inertial

File: src/turtle/urdf/turtle.urdf (robot description, URDF)
Before this commit: robot turtle, 5 links, 4 joints
Links:
- link base_link: mass None -> 1.0
- link front_caster: mass None -> 0.1
- link front_wheel: mass None -> 0.1
- link left_wheel: mass None -> 0.1; geometry collision cylinder length=0.05 radius=0.035; visual cylinder length=0.05 radius=0.035
- link right_wheel: mass None -> 0.1
