Commit message: Added laser scanner

File: src/turtle/urdf/turtle.urdf.xacro (robot description, xacro)
@@ -82,7 +82,61 @@
     <xacro:xtransmission name="trans2" motor_name="motor2" hardware_interface="VelocityJointInterface" joint="left_wheel_joint" />
     <xacro:xtransmission name="trans3" motor_name="motor3" hardware_interface="VelocityJointInterface" joint="right_wheel_joint" />
+    <!-- Laser -->
+    <link name="laser_link">
+        <collision>
+            <origin xyz="0 0 0" rpy="0 0 0" />
+            <geometry>
+                <box size="0.1 0.1 0.1" />
+            </geometry>
+        </collision>
+        <visual>
+            <origin xyz="0 0 0" rpy="0 0 0" />
+            <geometry>
+                <box size="0.1 0.1 0.1" />
+            </geometry>
+            <material name="laser_paint">
+                <color rgba="0.5 0.9 0.5 1.0" />
+            </material>
+        </visual>
+        <inertial>
+            <mass value="1e-5" />
+            <origin xyz="0 0 0" rpy="0 0 0" />
+            <inertia ixx="1e-6" ixy="0" ixz="0" iyy="1e-6" iyz="0" izz="1e-6" />
+        </inertial>
+    </link>
+    <joint name="laser_joint" type="fixed">
+        <axis xyz="0 1 0" />
+        <origin xyz="0 0 0.2" rpy="0 0 0" />
+        <parent link="front_caster" />
+        <child link="laser_link" />
+    </joint>
     <gazebo>
-        <plugin name="gazebo_ros_control" filename="libgazebo_ros_control.so">
-        </plugin>
+        <plugin name="gazebo_ros_control" filename="libgazebo_ros_control.so"></plugin>
+    </gazebo>
+    <gazebo reference="laser_link">
+        <sensor type="gpu_ray" name="laser">
+            <pose> 0 0 0 0 0 0</pose>
+            <visualize>false</visualize>
+            <update_rate>10</update_rate>
+            <ray>
+                <scan>
+                    <horizontal>
+                        <samples>300</samples>
+                        <resolution>1</resolution>
+                        <min_angle>-1.570796</min_angle>
+                        <max_angle>1.570796</max_angle>
+                    </horizontal>
+                </scan>
+                <range>
+                    <min>0.10</min>
+                    <max>30.0</max>
+                    <resolution>0.01</resolution>
+                </range>
+            </ray>
+            <plugin name="gpu_laser" filename="libgazebo_ros_gpu_laser.so">
+                <topicName>/laser_scan</topicName>
+                <frameName>laser_link</frameName>
+            </plugin>
+        </sensor>
     </gazebo>
 </robot>
